File: lime-gpio expander/lime_gpio expander.kicad_pcb (KiCad board)
At the start: 2 copper layers, 97.5 x 44.7 mm, 16 parts, among them P1 CONN_01X02

Commit message: I guess I should actually start comitting this stuff, huh. Maybe so it's not only on my computer. This adds most of my work on the 3 channel board. and all the work on the 16-channel one. and maybe some other stuff. I don't know.
Other:
- board text added: "David Lenfesty 2015"
- board text removed: "David Lenfesty, 2015"
Changed lines of the file:
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@@
     (links 120)
     (no_connects 0)
-    (area 105.735 67.381 210.648334 117.017762)
+    (area 105.735 66.873 210.140334 117.017762)
     (thickness 1.6)
     (drawings 9)
@@
   )
   (setup
-    (last_trace_width 0.508)
+    (last_trace_width 0.254)
     (user_trace_width 0.508)
     (trace_clearance 0.254)
@@
     (visible_elements FFFFFFBF)
     (pcbplotparams
-      (layerselection 0x00030_80000001)
-      (usegerberextensions true)
+      (layerselection 0x010f0_80000001)
+      (usegerberextensions false)
       (excludeedgelayer true)
       (linewidth 0.150000)
@@
       (outputformat 1)
       (mirror false)
-      (drillshape 1)
+      (drillshape 0)
       (scaleselection 1)
-      (outputdirectory ""))
+      (outputdirectory Gerbers/))
   )
   (net 0 "")
@@
     )
   )
-  (gr_text "David Lenfesty, 2015" (at 205.994 102.87 90) (layer F.SilkS)
+  (gr_text "David Lenfesty 2015" (at 205.994 102.87 90) (layer F.SilkS)
     (effects (font (size 1.5 1.5) (thickness 0.3)))
   )
@@
   (gr_line (start 207.264 71.12) (end 110.236 71.12) (angle 90) (layer Edge.Cuts) (width 0.1))
   (segment (start 199.39 78.232) (end 202.438 78.232) (width 0.508) (layer B.Cu) (net 1))
-  (segment (start 202.438 78.232) (end 204.978 75.692) (width 0.508) (layer B.Cu) (net 1) (status 800000))
+  (segment (start 202.438 78.232) (end 204.978 75.692) (width 0.508) (layer B.Cu) (net 1))
   (segment (start 144.272 108.712) (end 176.276 108.712) (width 0.508) (layer B.Cu) (net 1))
   (segment (start 176.276 108.712) (end 176.53 108.966) (width 0.508) (layer B.Cu) (net 1))
@@
   (segment (start 129.286 102.87) (end 130.81 102.87) (width 0.254) (layer F.Cu) (net 9))
   (segment (start 128.524 102.108) (end 129.286 102.87) (width 0.254) (layer F.Cu) (net 9))
-  (segment (start 199.39 113.284) (end 199.39 114.046) (width 0.508) (layer B.Cu) (net 10) (status C00000))
-  (segment (start 199.39 114.046) (end 198.374 115.062) (width 0.508) (layer B.Cu) (net 10) (status 400000))
-  (segment (start 168.148 115.062) (end 167.132 114.046) (width 0.508) (layer B.Cu) (net 10) (status 800000))
+  (segment (start 199.39 113.284) (end 199.39 114.046) (width 0.508) (layer B.Cu) (net 10))
+  (segment (start 199.39 114.046) (end 198.374 115.062) (width 0.508) (layer B.Cu) (net 10))
+  (segment (start 168.148 115.062) (end 167.132 114.046) (width 0.508) (layer B.Cu) (net 10))
   (segment (start 198.374 115.062) (end 168.148 115.062) (width 0.508) (layer B.Cu) (net 10))
-  (segment (start 167.132 114.046) (end 167.132 113.284) (width 0.508) (layer B.Cu) (net 10) (status C00000))
+  (segment (start 167.132 114.046) (end 167.132 113.284) (width 0.508) (layer B.Cu) (net 10))
   (segment (start 167.132 113.284) (end 167.132 113.792) (width 0.508) (layer B.Cu) (net 10))
   (segment (start 167.132 113.792) (end 165.862 115.062) (width 0.508) (layer B.Cu) (net 10))
