File: 3Channel-LED-Driver-NoSensing/3Channel-LED-Driver-NoSensing.sch (KiCad schematic (older format))
At the start: 3 parts, among them P2 CONN_01X02

Commit message: I guess I should actually start comitting this stuff, huh. Maybe so it's not only on my computer. This adds most of my work on the 3 channel board. and all the work on the 16-channel one. and maybe some other stuff. I don't know.
Parts:
- removed P2: CONN_01X02, symbol CONN_01X02
- removed P?: CONN_01X03, symbol CONN_01X03
- removed U?: PCA9633, symbol PCA9633
- added D1, D2, D3: LED, LEDs:LED-3MM, symbol LED
- added JP1, JP2: Jumper_NO_Small, Connect:GS2, symbol Jumper_NO_Small
- added P1, P7: CONN_01X02, Pin_Headers:Pin_Header_Straight_1x02, symbol CONN_01X02
- added P2, P4: CONN_01X03, Pin_Headers:Pin_Header_Straight_1x03, symbol CONN_01X03
- added P3: CONN_01X04, Pin_Headers:Pin_Header_Straight_1x04, symbol CONN_01X04
- added Q1, Q3, Q5: BUT11A, Power_Integrations:TO-220, symbol BUT11A
- added Q2, Q4, Q6, Q7, Q8, Q9: BC413, TO_SOT_Packages_THT:TO-92_Inline_Narrow_Oval, symbol BC413
- added R1, R4, R7: 10K, Resistors_ThroughHole:Resistor_Horizontal_RM7mm, symbol R
- added R10, R11: 4.7K, Resistors_ThroughHole:Resistor_Horizontal_RM7mm, symbol R
- added R12, R13, R14: 330, Resistors_ThroughHole:Resistor_Horizontal_RM7mm, symbol R
- added R15, R16, R17: 50K, Resistors_ThroughHole:Resistor_Horizontal_RM7mm, symbol R
- added R2, R5, R8: 2K, Resistors_ThroughHole:Resistor_Horizontal_RM7mm, symbol R
- added R3, R6, R9: R, Custom_Footprints:Current_Sense_Resistor, symbol R
- added RV1, RV2, RV3: 10K, Potentiometers:Potentiometer_VishaySpectrol-Econtrim-Type36P, symbol POT
- added U1: PCA9633, Housings_SSOP:TSSOP-10_3x3mm_Pitch0.5mm, symbol PCA9633
- added U2: LM324AN, Housings_DIP:DIP-14_W7.62mm, symbol LM324AN
Connections:
- net labels added: +3.3V, +5V, LED0_IND, LED1_IND, LED2_IND
- net labels removed: VCC
- wire segments 8 -> 90

Commit message: Finished most of the work on the 16 Channel LED driver, finished RevA at least. There are still a few vestigal folders to delete and stuff to clean, but I'm lazy.
Parts:
- D1, D2, D3: symbol LED -> LED-RESCUE-3Channel-LED-Driver-NoSensing
- RV1, RV2, RV3: symbol POT -> POT-RESCUE-3Channel-LED-Driver-NoSensing
Changed lines of the file:
@@
 EESchema Schematic File Version 2
+LIBS:3Channel-LED-Driver-NoSensing-rescue
 LIBS:power
 LIBS:device
@@
 $EndComp
 $Comp
-L POT RV1
+L POT-RESCUE-3Channel-LED-Driver-NoSensing RV1
 U 1 1 579912B6
 P 4700 2400
@@
 $EndComp
 $Comp
-L POT RV2
+L POT-RESCUE-3Channel-LED-Driver-NoSensing RV2
 U 1 1 57992148
 P 6750 2450
@@
 $EndComp
 $Comp
-L POT RV3
+L POT-RESCUE-3Channel-LED-Driver-NoSensing RV3
 U 1 1 579924B0
 P 9200 2450
@@
 $EndComp
 $Comp
-L LED D1
+L LED-RESCUE-3Channel-LED-Driver-NoSensing D1
 U 1 1 5799533D
 P 6400 4600
@@
 $EndComp
 $Comp
-L LED D3
+L LED-RESCUE-3Channel-LED-Driver-NoSensing D3
 U 1 1 579958DC
 P 6400 6950
@@
 $EndComp
 $Comp
-L LED D2
+L LED-RESCUE-3Channel-LED-Driver-NoSensing D2
 U 1 1 57995BEB
 P 6400 5750
