File: PCA9685_LED_Driver/PCA9685_LED_Driver.kicad_pcb (KiCad board)
At the start: 2 copper layers, 163 parts, among them P1 CONN_01X03, P2 CONN_01X02, P3 CONN_01X02, P4 CONN_01X02, P5 CONN_01X16, P6 CONN_01X16, Q1 BC413, Q10 BD911, Q11 BC413, Q12 BC413, Q13 BC413, Q14 BC413, Q15 BD911, Q16 BD911, Q17 BC413, Q18 BC413, Q19 BC413, Q2 BC413, Q20 BC413, Q21 BD911, Q22 BD911, Q23 BC413, Q24 BC413, Q25 BC413, Q26 BC413, Q27 BD911, Q28 BD911, Q29 BC413, Q3 BD911, Q30 BC413, Q31 BC413, Q32 BC413, Q33 BD911, Q34 BD911, Q35 BC413, Q36 BC413, Q37 BC413, Q38 BC413, Q39 BD911, Q4 BD911, Q40 BD911, Q41 BC413, Q42 BC413, Q43 BC413, Q44 BC413, Q45 BD911, Q46 BD911, Q47 BC413, Q48 BC413, Q5 BC413, Q6 BC413, Q7 BC413, Q8 BC413, Q9 BD911, U1 PCA9685, U2 LM324AN, U3 LM324AN, U4 LM324AN, U5 LM324AN

Commit message: Finished most of the work on the 16 Channel LED driver, finished RevA at least. There are still a few vestigal folders to delete and stuff to clean, but I'm lazy.
Parts:
- removed D6: LED, LEDs:LED_0805
- removed P4: CONN_01X02, Socket_Strips:Socket_Strip_Angled_1x02
- removed R1, R2: R, Resistors_SMD:R_0805_HandSoldering
- added C1: CP_Small, Capacitors_Tantalum_SMD:TantalC_SizeA_EIA-3216_HandSoldering, F.Cu at (56.9, 151.9)
- added C2: CP_Small, Capacitors_Tantalum_SMD:TantalC_SizeA_EIA-3216_HandSoldering, F.Cu at (47.8, 152.4)
- added P7: CONN_01X06, Custom_Footprints:Screw_Connector_M5, F.Cu at (65.8, 113.2)
- added Q49: BC413, TO_SOT_Packages_SMD:SOT-23, F.Cu at (274.8, 60.5)
- added Q50: BC413, TO_SOT_Packages_SMD:SOT-23, F.Cu at (33.5, 99.6)
- added Q51: BC413, TO_SOT_Packages_SMD:SOT-23, F.Cu at (291.1, 60.9)
- added Q52: BC413, TO_SOT_Packages_SMD:SOT-23, F.Cu at (23.9, 132.6)
- added Q53: BC413, TO_SOT_Packages_SMD:SOT-23, F.Cu at (307.3, 61.5)
- added Q54: BC413, TO_SOT_Packages_SMD:SOT-23, F.Cu at (167.1, 148.6)
- added Q55: BC413, TO_SOT_Packages_SMD:SOT-23, F.Cu at (323.1, 62.0)
- added Q56: BC413, TO_SOT_Packages_SMD:SOT-23, F.Cu at (73.2, 127.5)
- added Q57: BC413, TO_SOT_Packages_SMD:SOT-23, F.Cu at (78.2, 164.1)
- added Q58: BC413, TO_SOT_Packages_SMD:SOT-23, F.Cu at (60.5, 125.0)
- added Q59: BC413, TO_SOT_Packages_SMD:SOT-23, F.Cu at (77.2, 140.2)
- added Q60: BC413, TO_SOT_Packages_SMD:SOT-23, F.Cu at (25.4, 125.5)
- added Q61: BC413, TO_SOT_Packages_SMD:SOT-23, F.Cu at (34.0, 126.0)
- added Q62: BC413, TO_SOT_Packages_SMD:SOT-23, F.Cu at (34.5, 112.3)
- added Q63: BC413, TO_SOT_Packages_SMD:SOT-23, F.Cu at (42.7, 112.3)
- added Q64: BC413, TO_SOT_Packages_SMD:SOT-23, F.Cu at (47.8, 112.3)
- added U6: LD3985M47R, TO_SOT_Packages_SMD:SOT-23-5, F.Cu at (39.6, 150.9)
- P1: value CONN_01X03 -> CONN_01X02
- Q12, Q14, Q18, Q2, Q20, Q24, Q6, Q8: moved to B.Cu
- R10, R17, R18, R25, R26, R33, R34, R41, R42, R49, R50, R57, R58, R65, R66, R9: value Rsense -> 0.08
- R37, R45, R53, R61: value R -> 10K
- moved U3 303.6 mm to (474.1, 65.9)
- moved RV6 300.9 mm to (482.7, 67.6)
- moved RV8 299.2 mm to (482.7, 61.9)
- moved RV4 289.7 mm to (467.4, 67.6)
- moved R34 275.0 mm to (454.3, 77.7), turned to 270 degrees
- moved R20 272.5 mm to (474.9, 76.5), turned to 270 degrees
- moved Q16 271.9 mm to (438.9, 62.5), turned to 90 degrees
- moved Q22 271.9 mm to (454.6, 63.1), turned to 90 degrees
- moved RV2 269.5 mm to (467.4, 61.6)
- moved R28 267.8 mm to (477.4, 76.5), turned to 270 degrees
- moved D2 257.6 mm to (467.2, 72.9)
- moved Q10 256.1 mm to (422.6, 62.5), turned to 90 degrees
- moved D4 247.3 mm to (471.4, 72.9)
- moved R26 246.8 mm to (438.4, 77.5), turned to 270 degrees
- moved R12 242.1 mm to (472.3, 76.5), turned to 270 degrees
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Connections:
- P1 pad 1: +3V3 -> +5V
- P1 pad 2: +5V -> GND
- P1 pad 3: GND -> (no net)
Routing:
- net Net-(Q4-Pad3): track 0.00 -> 109.3 mm
- net Net-(Q10-Pad3): track 0.00 -> 95.4 mm
- net Net-(Q16-Pad3): track 0.00 -> 80.6 mm
- net Net-(Q14-Pad2): track 0.00 -> 52.8 mm, vias 0 -> 5
- net Net-(Q20-Pad2): track 0.00 -> 49.7 mm, vias 0 -> 3
- net Net-(Q22-Pad3): track 0.00 -> 47.5 mm
- net Net-(Q6-Pad2): track 0.00 -> 26.3 mm, vias 0 -> 1
- net Net-(Q24-Pad2): track 0.00 -> 25.1 mm, vias 0 -> 1
- net +5V: track 0.00 -> 24.3 mm, vias 0 -> 1
- net Net-(RV8-Pad2): track 0.00 -> 19.3 mm
- net Net-(Q18-Pad2): track 0.00 -> 19.1 mm, vias 0 -> 3
- net Net-(Q12-Pad2): track 0.00 -> 18.6 mm, vias 0 -> 3
- net Net-(RV2-Pad2): track 0.00 -> 17.2 mm
- net Net-(RV6-Pad2): track 0.00 -> 11.9 mm, vias 0 -> 2
- net Net-(P5-Pad8): track 0.00 -> 6.28 mm
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