File: PCA9685_LED_Driver/file57C20972.sch (KiCad schematic (older format))
At the start: 83 parts, among them P5 CONN_01X16, Q1 BC413, Q10 BD911, Q11 BC413, Q12 BC413, Q13 BC413, Q14 BC413, Q15 BD911, Q16 BD911, Q17 BC413, Q18 BC413, Q19 BC413, Q2 BC413, Q20 BC413, Q21 BD911, Q22 BD911, Q23 BC413, Q24 BC413, Q3 BD911, Q4 BD911, Q49 BC413, Q5 BC413, Q50 BC413, Q51 BC413, Q52 BC413, Q53 BC413, Q54 BC413, Q55 BC413, Q56 BC413, Q6 BC413, Q7 BC413, Q8 BC413, Q9 BD911, U2 LM324AN, U3 LM324AN

Commit message: Finished most of the work on the 16 Channel LED driver, finished RevA at least. There are still a few vestigal folders to delete and stuff to clean, but I'm lazy.
Parts:
- removed Q1, Q11, Q49, Q5, Q51: BC413, TO_SOT_Packages_SMD:SOT-23, symbol BC413
- D1, D2, D3, D4, D5, D6, D7, D8: symbol LED -> LED-RESCUE-PCA9685_LED_Driver
- R3: value 500 -> 499
- R5: value R -> 10K
- RV1, RV2, RV3, RV4, RV5, RV6, RV7, RV8: symbol POT -> POT-RESCUE-PCA9685_LED_Driver
Connections:
- net GND: no longer D1.1 (K)
- net LED0: now also R3.2
Other:
- moved on the sheet: D1, R3
