File: PCA9685_LED_Driver/file57C22724.sch (KiCad schematic (older format))
At the start: 83 parts, among them P6 CONN_01X16, Q25 BC413, Q26 BC413, Q27 BD911, Q28 BD911, Q29 BC413, Q30 BC413, Q31 BC413, Q32 BC413, Q33 BD911, Q34 BD911, Q35 BC413, Q36 BC413, Q37 BC413, Q38 BC413, Q39 BD911, Q40 BD911, Q41 BC413, Q42 BC413, Q43 BC413, Q44 BC413, Q45 BD911, Q46 BD911, Q47 BC413, Q48 BC413, Q57 BC413, Q58 BC413, Q59 BC413, Q60 BC413, Q61 BC413, Q62 BC413, Q63 BC413, Q64 BC413, U4 LM324AN, U5 LM324AN

Commit message: Finished most of the work on the 16 Channel LED driver, finished RevA at least. There are still a few vestigal folders to delete and stuff to clean, but I'm lazy.
Parts:
- D10, D11, D12, D13, D14, D15, D16, D9: symbol LED -> LED-RESCUE-PCA9685_LED_Driver
- RV10, RV11, RV12, RV13, RV14, RV15, RV16, RV9: symbol POT -> POT-RESCUE-PCA9685_LED_Driver
