File: stm32f030-eth/stm32f030-eth.kicad_pcb (KiCad board)
At the start: 2 copper layers, 62.5 x 53.5 mm, 47 parts, among them CON1 Micro_SD_Card, P1 CONN_01X06, P10 CONN_01X02, P11 CONN_01X02, P12 CONN_01X02, P13 CONN_01X02, P14 CNT-RJ45, P2 CONN_01X02, P3 CONN_01X02, P4 CONN_01X02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

Commit message: forgot a few silkscreen words
Other:
- board text added: "DUP"
- board text added: "SPD"
Changed lines of the file:
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@@
     (area 29.924999 19.924999 92.575001 73.575001)
     (thickness 1.6)
-    (drawings 62)
+    (drawings 64)
     (tracks 1387)
     (zones 0)
@@
     (36 B.SilkS user)
     (37 F.SilkS user)
-    (38 B.Mask user hide)
+    (38 B.Mask user)
     (39 F.Mask user hide)
-    (40 Dwgs.User user hide)
-    (41 Cmts.User user hide)
-    (42 Eco1.User user hide)
-    (43 Eco2.User user)
+    (40 Dwgs.User user)
+    (41 Cmts.User user)
+    (42 Eco1.User user)
+    (43 Eco2.User user hide)
     (44 Edge.Cuts user)
-    (45 Margin user hide)
+    (45 Margin user)
     (46 B.CrtYd user hide)
-    (47 F.CrtYd user hide)
-    (48 B.Fab user hide)
-    (49 F.Fab user hide)
+    (47 F.CrtYd user)
+    (48 B.Fab user)
+    (49 F.Fab user)
   )
   (setup
@@
     )
   )
-  (gr_text PA5 (at 87 61.5 360) (layer B.SilkS)
+  (gr_text SPD (at 72 42) (layer F.SilkS)
+    (effects (font (size 1.5 1.5) (thickness 0.3)))
+  )
+  (gr_text DUP (at 61.25 42) (layer F.SilkS)
+    (effects (font (size 1.5 1.5) (thickness 0.3)))
+  )
+  (gr_text PA5 (at 87 61.5) (layer B.SilkS)
     (effects (font (size 1.5 1.5) (thickness 0.3)) (justify mirror))
   )
-  (gr_text PA4 (at 86.75 53.5 360) (layer B.SilkS)
+  (gr_text PA4 (at 86.75 53.5) (layer B.SilkS)
     (effects (font (size 1.5 1.5) (thickness 0.3)) (justify mirror))
   )
-  (gr_text PA3 (at 86.75 45.75 360) (layer B.SilkS)
+  (gr_text PA3 (at 86.75 45.75) (layer B.SilkS)
     (effects (font (size 1.5 1.5) (thickness 0.3)) (justify mirror))
   )
-  (gr_text PA2 (at 86.75 38 360) (layer B.SilkS)
+  (gr_text PA2 (at 86.75 38) (layer B.SilkS)
     (effects (font (size 1.5 1.5) (thickness 0.3)) (justify mirror))
   )
-  (gr_text PA1 (at 86.5 29.75 360) (layer B.SilkS)
+  (gr_text PA1 (at 86.5 29.75) (layer B.SilkS)
     (effects (font (size 1.5 1.5) (thickness 0.3)) (justify mirror))
   )
-  (gr_text PA0 (at 86.5 22 360) (layer B.SilkS)
+  (gr_text PA0 (at 86.5 22) (layer B.SilkS)
     (effects (font (size 1.5 1.5) (thickness 0.3)) (justify mirror))
   )

Commit message: Fixed some errors in the 8p8c connector. Added a reset switch. Added a BOM
Parts:
- added C10: 0.1uF, Capacitors_SMD:C_0805_HandSoldering, F.Cu at (71.5, 66.8)
- added SW1: SW_Push, Buttons_Switches_SMD:SW_SPST_B3S-1000, F.Cu at (55.0, 65.5)
Routing:
- net /NRST: track 7.94 -> 32.0 mm, vias 0 -> 2
- net AGND: track 90.5 -> 98.5 mm, vias 27 -> 28
