File: stm32f030-eth/stm32f030-eth.sch (KiCad schematic (older format))
At the start: 47 parts, among them CON1 Micro_SD_Card, P1 CONN_01X06, P10 CONN_01X02, P11 CONN_01X02, P12 CONN_01X02, P13 CONN_01X02, P14 CNT-RJ45, P2 CONN_01X02, P3 CONN_01X02, P4 CONN_01X02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

Commit message: Fixed some errors in the 8p8c connector. Added a reset switch. Added a BOM
Parts:
- added C10: 0.1uF, Capacitors_SMD:C_0805_HandSoldering, symbol C
- added SW1: SW_Push, Buttons_Switches_SMD:SW_SPST_B3S-1000, symbol SW_Push
Connections:
- net GND: now also C10.2, SW1.1
- net NRST: now also C10.1, SW1.2
Changed lines of the file:
@@
 LIBS:w5500
 LIBS:stm32f030r8t6
+LIBS:switches
 LIBS:stm32f030-eth-cache
 EELAYER 25 0
@@
 	5550 5150 5450 5150
 Connection ~ 5450 5150
+$Comp
+L SW_Push SW1
+U 1 1 58D48FFE
+P 850 2450
+F 0 "SW1" H 900 2550 50  0000 L CNN
+F 1 "SW_Push" H 850 2390 50  0000 C CNN
+F 2 "Buttons_Switches_SMD:SW_SPST_B3S-1000" H 850 2650 50  0001 C CNN
+F 3 "" H 850 2650 50  0000 C CNN
+	1    850  2450
+	0    -1   -1   0
+$EndComp
+$Comp
+L C C10
+U 1 1 58D4933D
+P 1200 2400
+F 0 "C10" H 1225 2500 50  0000 L CNN
+F 1 "0.1uF" H 1225 2300 50  0000 L CNN
+F 2 "Capacitors_SMD:C_0805_HandSoldering" H 1238 2250 50  0001 C CNN
+F 3 "" H 1200 2400 50  0000 C CNN
+	1    1200 2400
+	1    0    0    -1
+$EndComp
+Wire Wire Line
+	850  2250 1450 2250
+Connection ~ 1450 2250
+Connection ~ 1200 2250
+Wire Wire Line
+	1200 2550 1200 2850
+$Comp
+L GND #PWR026
+U 1 1 58D49789
+P 1200 2850
+F 0 "#PWR026" H 1200 2600 50  0001 C CNN
+F 1 "GND" H 1200 2700 50  0000 C CNN
+F 2 "" H 1200 2850 50  0000 C CNN
+F 3 "" H 1200 2850 50  0000 C CNN
+	1    1200 2850
+	1    0    0    -1
+$EndComp
+$Comp
+L GND #PWR027
+U 1 1 58D49803
+P 850 2850
+F 0 "#PWR027" H 850 2600 50  0001 C CNN
+F 1 "GND" H 850 2700 50  0000 C CNN
+F 2 "" H 850 2850 50  0000 C CNN
+F 3 "" H 850 2850 50  0000 C CNN
+	1    850  2850
+	1    0    0    -1
+$EndComp
+Wire Wire Line
+	850  2650 850  2850
 $EndSCHEMATC
