File: Altoids-PowerSupply/Altoids-PowerSupply.sch (KiCad schematic (older format))
At the start: 47 parts, among them J1 Conn_01x04_Male, J10 USB_A, J2 Conn_01x04_Female, J3 Conn_01x04_Male, J4 Conn_01x04_Female, J5 Conn_01x04_Male, J6 Conn_01x04_Female, J7 Conn_01x06, J8 Conn_01x02, J9 USB_OTG, Q1 Q_PMOS_GDS, SW1 SW_DIP_x01, SW2 SW_DIP_x01, U1 MC34063, U2 MC34063, U3 KeyElco-1043P, U4 BQ24230, U5 AP2127K-3.3TRG1, U6 ATTINY45-20SU

Commit message: Rev A possibly complete, need to review to ensure no errors. Generated some preliminary gerbers to check things.
Parts:
- removed SW1: SW_DIP_x01, symbol SW_DIP_x01
- added C10, C9: Cfilter, Capacitors_SMD:CP_Elec_5x5.3, symbol CP
- added L3, L4: 1uH, Inductors_THT:L_Axial_L12.0mm_D5.0mm_P5.08mm_Vertical_Fastron_MISC, symbol L
- added R14: 10K, Resistors_SMD:R_0805_HandSoldering, symbol R
- added SW1: SW_Push, Buttons_Switches_SMD:SW_SPST_PTS810, symbol SW_Push
- C1, C4: value 100uH -> 100uF; footprint (none) -> Capacitors_SMD:CP_Elec_5x5.3; symbol C -> CP
- C2, C5, C7, C8: footprint (none) -> Capacitors_SMD:C_0805_HandSoldering
- C3, C6: footprint (none) -> Capacitors_SMD:CP_Elec_5x5.3; symbol C -> CP
- D1, D2: footprint (none) -> Diodes_SMD:D_0805
- D3, D4, D5: footprint (none) -> LEDs:LED_0805_HandSoldering
- J1, J3, J5: footprint (none) -> Pin_Headers:Pin_Header_Straight_1x04_Pitch2.54mm
- J10: footprint (none) -> Connectors:USB_A
- J2, J4, J6: footprint (none) -> Socket_Strips:Socket_Strip_Straight_1x04_Pitch2.54mm
- J7: footprint (none) -> Pin_Headers:Pin_Header_Straight_2x03_Pitch2.54mm
- J8: footprint (none) -> Pin_Headers:Pin_Header_Straight_1x02_Pitch2.54mm
- J9: footprint (none) -> Connectors:USB_Micro-B
- L1, L2: footprint (none) -> Inductors_THT:L_Radial_D9.5mm_P5.00mm_Fastron_07HVP
- Q1: footprint (none) -> TO_SOT_Packages_SMD:TO-263-2
- R1, R10, R11, R12, R13, R2, R3, R5, R7, R8, R9: footprint (none) -> Resistors_SMD:R_0805_HandSoldering
- R4, R6: footprint (none) -> Resistors_SMD:R_1206_HandSoldering
- SW2: footprint (none) -> Buttons_Switches_SMD:SW_DIP_x1_W5.08mm_Slide_Copal_CHS-A
- U1, U2: footprint (none) -> Housings_SOIC:SOIC-8_3.9x4.9mm_Pitch1.27mm
- U3: footprint (none) -> cust_footprints:KeyElco-1043P
- U4: footprint (none) -> Housings_DFN_QFN:QFN-16-1EP_3x3mm_Pitch0.5mm_ThermalVias
- U5: footprint (none) -> TO_SOT_Packages_SMD:SOT-23-5
Connections:
- net GNDA is gone; now on net Earth: C1.2, C3.2, C4.2, C6.2, C7.2, C8.2, J1.3 (Pin_3), J1.4 (Pin_4), J2.3 (Pin_3), J2.4 (Pin_4), J3.3 (Pin_3), J3.4 (Pin_4), J4.3 (Pin_3), J4.4 (Pin_4), J5.3 (Pin_3), J5.4 (Pin_4), J6.3 (Pin_3), J6.4 (Pin_4), R1.2, R10.2, R11.2, R12.2, R13.2, R8.2, U4.17 (PAD), U4.5 (EN2), U4.8 (VSS), U5.2 (GND)
- net +12V: now also C10.1, L4.1; no longer C6.1, D2.1 (K), R7.1
- net +5V: now also J10.1 (VBUS), C9.1, L3.1; no longer C3.1, D1.1 (K), R2.1
- net Cutoff: no longer D3.2 (A), U6.2 (PB3(XTAL1/CLKI/~OC1B~/ADC3/PCINT3))
- net Earth: now also C10.2, C9.2, R14.2
- net OUT: now also Q1.2 (D)
- net SCK: now also SW1.2
- net PGOOD: now reaches D4.2 (A), U4.7 (~PGOOD)
- net CHG: now reaches D5.2 (A), U4.9 (~CHG)
- new net: C3.1, D1.1 (K), L3.2, R2.1
- new net: C6.1, D2.1 (K), L4.2, R7.1
- new net: R14.1, SW1.1
- new net IND: D3.2 (A), U6.2 (PB3(XTAL1/CLKI/~OC1B~/ADC3/PCINT3))
Other:
- note added: "Rsc = 0.24\nCt = 100pF\nL = 22uH\nCo = 330uF\nR1 = 10K\nR2 = 30K\nLfilter = 1uH\nCfilter = 100uF"
- note added: "Rsc = 0.33\nCt = 100pF\nL = 22uH\nCo = 47uF\nR1 = 1.5K\nR2 = 13K\nLfilter = 1uH\nCfilter = 100uF"
- note removed: "CHANGE THESE!!!"
- note removed: "Rsc = 0.24\nCt = 100pF\nL = 10uH\nCo = 330uF\nR1 = 10K\nR2 = 30K\nLfilter = 1uH\nCfilter = 100uF"
- note removed: "Rsc = 0.33\nCt = 100pF\nL = 18uH\nCo = 47uF\nR1 = 1.5K\nR2 = 13K\nLfilter = 1uH\nCfilter = 100uF"
