File: Altoids-PowerSupply/Altoids-PowerSupply.kicad_pcb (KiCad board)
At the start: 2 copper layers, 90.5 x 56 mm, 0 parts

Commit message: Rev A possibly complete, need to review to ensure no errors. Generated some preliminary gerbers to check things.
Parts:
- added C1: 100uF, Capacitors_SMD:CP_Elec_5x5.3, F.Cu at (123.5, 72.3)
- added C10: Cfilter, Capacitors_SMD:CP_Elec_5x5.3, F.Cu at (158.5, 82.5)
- added C2: Ct, Capacitors_SMD:C_0805_HandSoldering, B.Cu at (125.5, 73.8)
- added C3: Co, Capacitors_SMD:CP_Elec_5x5.3, F.Cu at (152.0, 75.0)
- added C4: 100uF, Capacitors_SMD:CP_Elec_5x5.3, F.Cu at (123.5, 84.5)
- added C5: Ct, Capacitors_SMD:C_0805_HandSoldering, B.Cu at (126.0, 85.2)
- added C6: Co, Capacitors_SMD:CP_Elec_5x5.3, F.Cu at (152.5, 87.0)
- added C7: 1uF, Capacitors_SMD:C_0805_HandSoldering, F.Cu at (125.5, 96.8)
- added C8: 1uF, Capacitors_SMD:C_0805_HandSoldering, F.Cu at (125.5, 90.8)
- added C9: Cfilter, Capacitors_SMD:CP_Elec_5x5.3, F.Cu at (158.5, 69.5)
- added D1: 1N5819, Diodes_SMD:D_0805, F.Cu at (145.9, 75.5)
- added D2: 1N5819, Diodes_SMD:D_0805, F.Cu at (145.9, 87.5)
- added D3: LED, LEDs:LED_0805_HandSoldering, F.Cu at (104.0, 92.8)
- added D4: LED, LEDs:LED_0805_HandSoldering, F.Cu at (109.5, 92.8)
- added D5: LED, LEDs:LED_0805_HandSoldering, F.Cu at (106.8, 92.8)
- added J1: Conn_01x04_Male, Pin_Headers:Pin_Header_Straight_1x04_Pitch2.54mm, F.Cu at (154.2, 95.8)
- added J10: USB_A, Connectors:USB_A, F.Cu at (163.5, 77.5)
- added J2: Conn_01x04_Female, Socket_Strips:Socket_Strip_Straight_1x04_Pitch2.54mm, F.Cu at (154.2, 91.8)
- added J3: Conn_01x04_Male, Pin_Headers:Pin_Header_Straight_1x04_Pitch2.54mm, F.Cu at (166.2, 85.7)
- added J4: Conn_01x04_Female, Socket_Strips:Socket_Strip_Straight_1x04_Pitch2.54mm, F.Cu at (162.2, 85.7)
- added J5: Conn_01x04_Male, Pin_Headers:Pin_Header_Straight_1x04_Pitch2.54mm, F.Cu at (139.3, 95.8)
- added J6: Conn_01x04_Female, Socket_Strips:Socket_Strip_Straight_1x04_Pitch2.54mm, F.Cu at (139.3, 91.8)
- added J7: Conn_01x06, Pin_Headers:Pin_Header_Straight_2x03_Pitch2.54mm, F.Cu at (95.4, 78.3)
- added J8: Conn_01x02, Pin_Headers:Pin_Header_Straight_1x02_Pitch2.54mm, F.Cu at (89.4, 80.8)
- added J9: USB_OTG, Connectors:USB_Micro-B, F.Cu at (90.0, 71.0)
- added L1: L, Inductors_THT:L_Radial_D9.5mm_P5.00mm_Fastron_07HVP, F.Cu at (140.0, 73.5)
- added L2: L, Inductors_THT:L_Radial_D9.5mm_P5.00mm_Fastron_07HVP, F.Cu at (140.0, 81.0)
- added L3: 1uH, Inductors_THT:L_Axial_L12.0mm_D5.0mm_P5.08mm_Vertical_Fastron_MISC, F.Cu at (152.0, 69.0)
- added L4: 1uH, Inductors_THT:L_Axial_L12.0mm_D5.0mm_P5.08mm_Vertical_Fastron_MISC, F.Cu at (152.0, 81.0)
- added Q1: Q_PMOS_GDS, TO_SOT_Packages_SMD:TO-263-2, F.Cu at (114.2, 73.6)
- added R1: R1, Resistors_SMD:R_0805_HandSoldering, B.Cu at (130.0, 73.3)
- added R10: 10K, Resistors_SMD:R_0805_HandSoldering, F.Cu at (104.5, 74.0)
- added R11: ISET, Resistors_SMD:R_0805_HandSoldering, F.Cu at (102.5, 74.0)
- added R12: 499, Resistors_SMD:R_0805_HandSoldering, B.Cu at (109.4, 94.8)
- added R13: 499, Resistors_SMD:R_0805_HandSoldering, B.Cu at (106.8, 94.8)
- added R14: 10K, Resistors_SMD:R_0805_HandSoldering, F.Cu at (113.6, 86.4)
- added R2: R2, Resistors_SMD:R_0805_HandSoldering, B.Cu at (132.5, 73.3)
- added R3: 180, Resistors_SMD:R_0805_HandSoldering, B.Cu at (127.5, 73.3)
- added R4: Rsc, Resistors_SMD:R_1206_HandSoldering, F.Cu at (130.0, 69.0)
- added R5: 180, Resistors_SMD:R_0805_HandSoldering, B.Cu at (129.0, 85.3)
- added R6: Rsc, Resistors_SMD:R_1206_HandSoldering, F.Cu at (129.0, 81.0)
- added R7: R2, Resistors_SMD:R_0805_HandSoldering, B.Cu at (133.0, 85.3)
- added R8: R1, Resistors_SMD:R_0805_HandSoldering, B.Cu at (131.0, 85.3)
- added R9: 499, Resistors_SMD:R_0805_HandSoldering, B.Cu at (104.0, 94.7)
- added SW1: SW_Push, Buttons_Switches_SMD:SW_SPST_PTS810, F.Cu at (116.2, 92.0)
- added SW2: SW_DIP_x01, Buttons_Switches_SMD:SW_DIP_x1_W5.08mm_Slide_Copal_CHS-A, F.Cu at (102.6, 84.2)
- added U1: MC34063, Housings_SOIC:SOIC-8_3.9x4.9mm_Pitch1.27mm, F.Cu at (130.5, 73.5)
- added U2: MC34063, Housings_SOIC:SOIC-8_3.9x4.9mm_Pitch1.27mm, F.Cu at (131.0, 85.5)
- added U3: KeyElco-1043P, cust_footprints:KeyElco-1043P, F.Cu at (131.0, 54.0)
- added U4: BQ24230, Housings_DFN_QFN:QFN-16-1EP_3x3mm_Pitch0.5mm_ThermalVias, F.Cu at (102.2, 68.0)
- added U5: AP2127K-3.3TRG1, TO_SOT_Packages_SMD:SOT-23-5, F.Cu at (125.2, 93.8)
- added U6: ATTINY45-20SU, Housings_SOIC:SOIC-8_3.9x4.9mm_Pitch1.27mm, F.Cu at (96.8, 90.4)
Routing:
- net Net-(C1-Pad1): track 0.00 -> 76.6 mm
- net BAT: track 0.00 -> 72.5 mm
- net +5V: track 0.00 -> 70.9 mm
- net Earth: track 0.00 -> 69.2 mm, vias 0 -> 24
- net OUT: track 0.00 -> 58.7 mm, vias 0 -> 2
- net /SCK: track 0.00 -> 40.6 mm
- net Net-(D2-Pad2): track 0.00 -> 35.6 mm
- net Net-(L2-Pad2): track 0.00 -> 34.8 mm, vias 0 -> 1
- net /MISO: track 0.00 -> 34.7 mm, vias 0 -> 5
- net Net-(D1-Pad2): track 0.00 -> 32.8 mm
- net Net-(L1-Pad2): track 0.00 -> 31.1 mm, vias 0 -> 1
- net +3V3: track 0.00 -> 31.1 mm
- net /PGOOD: track 0.00 -> 29.5 mm, vias 0 -> 4
- net Cutoff: track 0.00 -> 28.7 mm, vias 0 -> 1
- net +12V: track 0.00 -> 27.2 mm
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- added copper zone on B.Cu, net Earth
Other:
- board text added: "CHG"
- board text added: "IND"
- board text added: "PWR"

Commit message: Finished Revision A. Exported gerbers.
Routing:
- net Net-(C3-Pad1): track 10.2 -> 25.9 mm
- net Net-(J10-Pad2): track 0.00 -> 2.03 mm
- net Earth: track 69.2 -> 71.0 mm, vias 24 -> 25
Other:
- board text added: "2017"
- board text added: "David Lenfesty"
- board text added: "Rev A"
Changed lines of the file:
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@@
   (general
     (links 141)
-    (no_connects 12)
+    (no_connects 0)
     (area 84.015 41.899999 197.35 109.200001)
     (thickness 1.6)
-    (drawings 13)
-    (tracks 444)
+    (drawings 16)
+    (tracks 456)
     (zones 0)
     (modules 52)
@@
     )
   )
+  (gr_text "Rev A" (at 116.4 96.5) (layer F.SilkS)
+    (effects (font (size 1.5 1.5) (thickness 0.3)))
+  )
+  (gr_text 2017 (at 87.6 62.4 90) (layer F.SilkS)
+    (effects (font (size 1.5 1.5) (thickness 0.3)))
+  )
+  (gr_text "David Lenfesty" (at 90.1 57.2 90) (layer F.SilkS)
+    (effects (font (size 1.5 1.5) (thickness 0.3)))
+  )
   (gr_text "PWR\n" (at 109.5 88 90) (layer F.SilkS)
     (effects (font (size 1.5 1.5) (thickness 0.3)))
@@
   (segment (start 123.5 82.3) (end 125.7 82.3) (width 1) (layer F.Cu) (net 1))
   (segment (start 125.7 82.3) (end 127 81) (width 1) (layer F.Cu) (net 1))
+  (segment (start 91.35 72.3) (end 89.6 72.3) (width 0.25) (layer F.Cu) (net 2))
+  (via (at 89.6 72.3) (size 0.6) (drill 0.4) (layers F.Cu B.Cu) (net 2))
   (segment (start 128.3 84.865) (end 130.135 84.865) (width 0.25) (layer F.Cu) (net 2))
   (segment (start 130.135 84.865) (end 131 84) (width 0.25) (layer F.Cu) (net 2))
@@
   (via (at 99.5 91.035) (size 0.6) (drill 0.4) (layers F.Cu B.Cu) (net 14))
   (via (at 97.4 91) (size 0.6) (drill 0.4) (layers F.Cu B.Cu) (net 14))
+  (segment (start 108.1 72.675) (end 111.475 72.675) (width 0.75) (layer F.Cu) (net 15))
+  (segment (start 103.300308 70.42501) (end 103.400327 70.324991) (width 0.75) (layer F.Cu) (net 15))
+  (segment (start 105.900006 70.475006) (end 108.1 72.675) (width 0.75) (layer F.Cu) (net 15))
+  (segment (start 104.070017 70.475006) (end 105.900006 70.475006) (width 0.75) (layer F.Cu) (net 15))
+  (segment (start 103.920002 70.324991) (end 104.070017 70.475006) (width 0.75) (layer F.Cu) (net 15))
+  (segment (start 102.699692 70.42501) (end 103.300308 70.42501) (width 0.75) (layer F.Cu) (net 15))
+  (segment (start 102.674682 70.4) (end 102.699692 70.42501) (width 0.75) (layer F.Cu) (net 15))
+  (segment (start 103.400327 70.324991) (end 103.920002 70.324991) (width 0.75) (layer F.Cu) (net 15))
   (segment (start 92.4 82.7) (end 92.4 89.81) (width 0.25) (layer F.Cu) (net 15))
   (segment (start 92.4 89.81) (end 93.625 91.035) (width 0.25) (layer F.Cu) (net 15))
@@
   (segment (start 96.764999 77.084999) (end 97.090001 77.410001) (width 0.25) (layer F.Cu) (net 15))
   (segment (start 97.090001 77.410001) (end 97.94 78.26) (width 0.25) (layer F.Cu) (net 15))
-  (segment (start 108.1 72.675) (end 111.475 72.675) (width 0.75) (layer F.Cu) (net 15))
-  (segment (start 105.900001 70.475001) (end 108.1 72.675) (width 0.75) (layer F.Cu) (net 15))
-  (segment (start 102.749683 70.475001) (end 105.900001 70.475001) (width 0.75) (layer F.Cu) (net 15))
-  (segment (start 102.674682 70.4) (end 102.749683 70.475001) (width 0.75) (layer F.Cu) (net 15))
   (segment (start 102.2 70.8) (end 97.94 75.06) (width 0.25) (layer F.Cu) (net 15))
   (segment (start 97.94 75.06) (end 97.94 78.26) (width 0.25) (layer F.Cu) (net 15))
@@
   (segment (start 95.4 87.67) (end 94.575 88.495) (width 0.25) (layer F.Cu) (net 17))
   (segment (start 94.575 88.495) (end 94.1 88.495) (width 0.25) (layer F.Cu) (net 17))
+  (via (at 103.675026 69.449977) (size 0.6) (drill 0.4) (layers F.Cu B.Cu) (net 18))
+  (segment (start 103.425049 69.2) (end 103.675026 69.449977) (width 0.25) (layer B.Cu) (net 18))
+  (segment (start 103.725 68.75) (end 103.725 69.400003) (width 0.25) (layer F.Cu) (net 18))
+  (segment (start 99.4 69.2) (end 103.425049 69.2) (width 0.25) (layer B.Cu) (net 18))
+  (segment (start 103.725 69.400003) (end 103.675026 69.449977) (width 0.25) (layer F.Cu) (net 18))
   (segment (start 99.4 69.2) (end 99.4 68) (width 0.25) (layer F.Cu) (net 18))
   (segment (start 99.4 68) (end 99.65 67.75) (width 0.25) (layer F.Cu) (net 18))
-  (segment (start 99.4 69.4) (end 99.4 69.2) (width 0.25) (layer B.Cu) (net 18))
-  (segment (start 99.6 69.6) (end 99.4 69.4) (width 0.25) (layer B.Cu) (net 18))
   (via (at 99.4 69.2) (size 0.6) (drill 0.4) (layers F.Cu B.Cu) (net 18))
-  (segment (start 103.65 69.6) (end 99.6 69.6) (width 0.25) (layer B.Cu) (net 18))
-  (segment (start 103.725 68.75) (end 103.725 69.525) (width 0.25) (layer F.Cu) (net 18))
-  (segment (start 103.725 69.525) (end 103.65 69.6) (width 0.25) (layer F.Cu) (net 18))
-  (via (at 103.65 69.6) (size 0.6) (drill 0.4) (layers F.Cu B.Cu) (net 18))
   (segment (start 92.8 69.6) (end 92.7 69.7) (width 0.5) (layer F.Cu) (net 18))
   (segment (start 92.7 69.7) (end 91.35 69.7) (width 0.5) (layer F.Cu) (net 18))
@@
   (segment (start 99.65 67.75) (end 95.45 67.75) (width 1) (layer F.Cu) (net 18))
   (segment (start 100.775 67.75) (end 99.65 67.75) (width 0.25) (layer F.Cu) (net 18))
+  (segment (start 163.5 75) (end 163.5 72.97) (width 0.25) (layer F.Cu) (net 22))
   (segment (start 129.424264 73.5) (end 129 73.5) (width 0.25) (layer F.Cu) (net 23))
   (segment (start 131.54 73.5) (end 129.424264 73.5) (width 0.25) (layer F.Cu) (net 23))
@@
   (segment (start 131.705 87.405) (end 131 86.7) (width 0.25) (layer F.Cu) (net 28))
   (via (at 131 86.7) (size 0.6) (drill 0.4) (layers F.Cu B.Cu) (net 28))
-  (segment (start 105.4 67.2) (end 104.725 66.525) (width 0.25) (layer F.Cu) (net 29))
-  (segment (start 104.725 66.525) (end 103 66.525) (width 0.25) (layer F.Cu) (net 29))
-  (segment (start 105.4 69.6) (end 105.4 67.2) (width 0.25) (layer F.Cu) (net 29))
-  (segment (start 105.2 71.4) (end 105.2 69.8) (width 0.25) (layer B.Cu) (net 29))
-  (segment (start 105.2 69.8) (end 105.4 69.6) (width 0.25) (layer B.Cu) (net 29))
-  (via (at 105.4 69.6) (size 0.6) (drill 0.4) (layers F.Cu B.Cu) (net 29))
+  (segment (start 105.2 71.4) (end 105.2 69.801226) (width 0.25) (layer B.Cu) (net 29))
+  (segment (start 105.401221 67.201221) (end 105.401221 69.175741) (width 0.25) (layer F.Cu) (net 29))
+  (segment (start 104.725 66.525) (end 105.401221 67.201221) (width 0.25) (layer F.Cu) (net 29))
+  (segment (start 105.401221 69.175741) (end 105.401221 69.600005) (width 0.25) (layer F.Cu) (net 29))
+  (via (at 105.401221 69.600005) (size 0.6) (drill 0.4) (layers F.Cu B.Cu) (net 29))
+  (segment (start 105.2 69.801226) (end 105.401221 69.600005) (width 0.25) (layer B.Cu) (net 29))
+  (segment (start 103 66.525) (end 104.725 66.525) (width 0.25) (layer F.Cu) (net 29))
   (segment (start 104.5 72.65) (end 104.5 72.1) (width 0.25) (layer F.Cu) (net 29))
   (segment (start 104.5 72.1) (end 105.2 71.4) (width 0.25) (layer F.Cu) (net 29))
   (via (at 105.2 71.4) (size 0.6) (drill 0.4) (layers F.Cu B.Cu) (net 29))
-  (segment (start 104.42501 67.553245) (end 104.121765 67.25) (width 0.25) (layer F.Cu) (net 30))
-  (segment (start 104.42501 69.000746) (end 104.42501 67.553245) (width 0.25) (layer F.Cu) (net 30))
-  (segment (start 104.6 69.175736) (end 104.42501 69.000746) (width 0.25) (layer F.Cu) (net 30))
-  (segment (start 104.6 69.6) (end 104.6 69.175736) (width 0.25) (layer F.Cu) (net 30))
-  (segment (start 104.121765 67.25) (end 103.725 67.25) (width 0.25) (layer F.Cu) (net 30))
-  (segment (start 104.2 71.4) (end 104.2 70) (width 0.25) (layer B.Cu) (net 30))
-  (segment (start 104.2 70) (end 104.6 69.6) (width 0.25) (layer B.Cu) (net 30))
-  (via (at 104.6 69.6) (size 0.6) (drill 0.4) (layers F.Cu B.Cu) (net 30))
-  (segment (start 102.5 72.65) (end 103.75 71.4) (width 0.25) (layer F.Cu) (net 30))
-  (segment (start 103.75 71.4) (end 104.2 71.4) (width 0.25) (layer F.Cu) (net 30))
-  (via (at 104.2 71.4) (size 0.6) (drill 0.4) (layers F.Cu B.Cu) (net 30))
+  (segment (start 103.411948 70.86861) (end 103.411948 71.292874) (width 0.25) (layer B.Cu) (net 30))
+  (segment (start 103.411948 70.78568) (end 103.411948 70.86861) (width 0.25) (layer B.Cu) (net 30))
+  (segment (start 104.601218 69.59641) (end 103.411948 70.78568) (width 0.25) (layer B.Cu) (net 30))
+  (segment (start 103.411948 71.638052) (end 103.411948 71.292874) (width 0.25) (layer F.Cu) (net 30))
+  (segment (start 104.35 67.25) (end 104.601218 67.501218) (width 0.25) (layer F.Cu) (net 30))
+  (segment (start 102.5 72.55) (end 103.411948 71.638052) (width 0.25) (layer F.Cu) (net 30))
+  (segment (start 102.5 72.65) (end 102.5 72.55) (width 0.25) (layer F.Cu) (net 30))
+  (via (at 103.411948 71.292874) (size 0.6) (drill 0.4) (layers F.Cu B.Cu) (net 30))
+  (segment (start 103.725 67.25) (end 104.35 67.25) (width 0.25) (layer F.Cu) (net 30))
+  (segment (start 104.601218 69.172146) (end 104.601218 69.59641) (width 0.25) (layer F.Cu) (net 30))
+  (segment (start 104.601218 67.501218) (end 104.601218 69.172146) (width 0.25) (layer F.Cu) (net 30))
+  (via (at 104.601218 69.59641) (size 0.6) (drill 0.4) (layers F.Cu B.Cu) (net 30))
   (segment (start 102 65.6) (end 102.6 65.6) (width 0.5) (layer F.Cu) (net 31))
   (segment (start 102 65.9) (end 102 65.6) (width 0.25) (layer F.Cu) (net 31))
@@
   (segment (start 102.6 65.6) (end 102.8 65.6) (width 0.25) (layer F.Cu) (net 31))
   (segment (start 102.5 66.525) (end 102.5 65.7) (width 0.25) (layer F.Cu) (net 31))
+  (segment (start 136.4 71) (end 144.92 71) (width 0.25) (layer B.Cu) (net 36))
+  (segment (start 144.92 71) (end 146.92 69) (width 0.25) (layer B.Cu) (net 36))
+  (segment (start 135.4 72) (end 136.4 71) (width 0.25) (layer B.Cu) (net 36))
+  (segment (start 132.5 72) (end 135.4 72) (width 0.25) (layer B.Cu) (net 36))
   (segment (start 147 75.5) (end 149.3 75.5) (width 1) (layer F.Cu) (net 36))
   (segment (start 149.3 75.5) (end 149.8 75) (width 1) (layer F.Cu) (net 36))

Commit message: Started Rev B of Altoids PSU.
Other:
- board text added: "12V"
- board text added: "3v3"
- board text added: "5V"
- board text added: "GND"
- board text added: "MISO"
- board text added: "MOSI"
- board text added: "RES"
- board text added: "Rev B"
- board text added: "SCK"
- board text added: "VTG"
- board text removed: "Rev A"
Changed lines of the file:
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@@
     (area 84.015 41.899999 197.35 109.200001)
     (thickness 1.6)
-    (drawings 16)
+    (drawings 33)
     (tracks 456)
     (zones 0)
@@
     (descr "Through hole straight pin header, 1x04, 2.54mm pitch, single row")
     (tags "Through hole pin header THT 1x04 2.54mm single row")
-    (fp_text reference J1 (at 0 -2.33 270) (layer F.SilkS)
+    (fp_text reference J1 (at 0.65 -2.45 270) (layer F.SilkS)
       (effects (font (size 1 1) (thickness 0.15)))
     )
@@
     (tags "resistor 0805")
     (attr smd)
-    (fp_text reference R10 (at 3.75 0 270) (layer F.SilkS)
+    (fp_text reference R10 (at 3.8 -0.7 270) (layer F.SilkS)
       (effects (font (size 1 1) (thickness 0.15)))
     )
@@
     (tags "resistor 0805")
     (attr smd)
-    (fp_text reference R11 (at 3.75 0 270) (layer F.SilkS)
+    (fp_text reference R11 (at 3.8 -0.9 270) (layer F.SilkS)
       (effects (font (size 1 1) (thickness 0.15)))
     )
@@
     (descr "Through hole straight socket strip, 1x04, 2.54mm pitch, single row")
     (tags "Through hole socket strip THT 1x04 2.54mm single row")
-    (fp_text reference J2 (at 0 -2.33 270) (layer F.SilkS)
+    (fp_text reference J2 (at -0.75 -2.35 270) (layer F.SilkS)
       (effects (font (size 1 1) (thickness 0.15)))
     )
@@
     (descr "Through hole straight pin header, 1x04, 2.54mm pitch, single row")
     (tags "Through hole pin header THT 1x04 2.54mm single row")
-    (fp_text reference J5 (at 0 -2.33 270) (layer F.SilkS)
+    (fp_text reference J5 (at 1.05 -2.47 270) (layer F.SilkS)
       (effects (font (size 1 1) (thickness 0.15)))
     )
@@
     (descr "Through hole straight socket strip, 1x04, 2.54mm pitch, single row")
     (tags "Through hole socket strip THT 1x04 2.54mm single row")
-    (fp_text reference J6 (at 0.25 -2.17 270) (layer F.SilkS)
+    (fp_text reference J6 (at -1.15 -2.37 270) (layer F.SilkS)
       (effects (font (size 1 1) (thickness 0.15)))
     )
@@
     )
   )
-  (gr_text "Rev A" (at 116.4 96.5) (layer F.SilkS)
+  (gr_text GND (at 89.4 85.5) (layer F.SilkS)
+    (effects (font (size 1 1) (thickness 0.25)))
+  )
+  (gr_text VTG (at 87.2 80.8 90) (layer F.SilkS)
+    (effects (font (size 1 1) (thickness 0.25)))
+  )
+  (gr_text MOSI (at 101.3 80) (layer F.SilkS)
+    (effects (font (size 1 1) (thickness 0.25)))
+  )
+  (gr_text VTG (at 100.8 78.2) (layer F.SilkS)
+    (effects (font (size 1 1) (thickness 0.25)))
+  )
+  (gr_text GND (at 98 85.6) (layer F.SilkS)
+    (effects (font (size 1 1) (thickness 0.25)))
+  )
+  (gr_text RES (at 92.6 83.5) (layer F.SilkS)
+    (effects (font (size 1 1) (thickness 0.25)))
+  )
+  (gr_text SCK (at 92.5 80.9) (layer F.SilkS)
+    (effects (font (size 1 1) (thickness 0.25)))
+  )
+  (gr_text MISO (at 92.3 78.3) (layer F.SilkS)
+    (effects (font (size 1 1) (thickness 0.25)))
+  )
+  (gr_line (start 160.5 89.5) (end 168.1 89.5) (layer F.SilkS) (width 0.2))
+  (gr_line (start 135.4 89.6) (end 135.4 97.7) (layer F.SilkS) (width 0.2))
+  (gr_line (start 150.4 90) (end 150.4 97.4) (layer F.SilkS) (width 0.2))
+  (gr_text 12V (at 171.9 85.8) (layer F.SilkS)
     (effects (font (size 1.5 1.5) (thickness 0.3)))
   )
+  (gr_text 5V (at 157.1 93.6 90) (layer F.SilkS)
+    (effects (font (size 1.5 1.5) (thickness 0.3)))
+  )
+  (gr_text 3v3 (at 141.8 93.7 90) (layer F.SilkS)
+    (effects (font (size 1.5 1.5) (thickness 0.3)))
+  )
+  (gr_text GND (at 164.1 95.7) (layer F.SilkS)
+    (effects (font (size 1.5 1.5) (thickness 0.3)))
+  )
+  (gr_text GND (at 129.5 93.6 90) (layer F.SilkS)
+    (effects (font (size 1.5 1.5) (thickness 0.3)))
+  )
+  (gr_text GND (at 144.4 93.7 90) (layer F.SilkS)
+    (effects (font (size 1.5 1.5) (thickness 0.3)))
+  )
+  (gr_text "Rev B" (at 116.4 96.5) (layer F.SilkS)
+    (effects (font (size 1.5 1.5) (thickness 0.3)))
+  )
