File: AC-LED-Control/_saved_AC-LED-Control.sch (KiCad schematic (older format))
At the start: 20 parts, among them P101 CONN_01X02, P102 CONN_01X02, P103 CONN_01X04, SW101 SW_PUSH, U101 FOD814-D, U102 STM32F030F4P6, U103 74HC595, U104 74HC595

Commit message: more stuff
Parts:
- gave numbers to parts that had none: 1
Changed lines of the file:
@@
 	650  7500 650  6300
 $Comp
-L CONN_01X02 P?
+L CONN_01X02 P104
 U 1 1 5B47C991
 P 5500 5200
-F 0 "P?" H 5500 5350 50  0000 C CNN
+F 0 "P104" H 5500 5350 50  0000 C CNN
 F 1 "CONN_01X02" V 5600 5200 50  0000 C CNN
 F 2 "" H 5500 5200 50  0000 C CNN
