File: AC-LED-Control/AC-LED-Control.kicad_pcb (KiCad board)
At the start: 4 copper layers, 139 parts, among them J101 Conn_01x03, J102 Conn_01x03, J103 Conn_01x02, J201 Conn_01x02, J202 Conn_01x02, J203 Conn_01x02, J204 Conn_01x02, J205 Conn_01x02, J206 Conn_01x02, J207 Conn_01x02, J208 Conn_01x02, J301 Conn_01x02, J302 Conn_01x02, J303 Conn_01x02, J304 Conn_01x02, J305 Conn_01x02, J306 Conn_01x02, J307 Conn_01x02, J308 Conn_01x02, P103 CONN_01X04, P104 CONN_01X02, P105 CONN_01X02, SW101 SW_PUSH, U101 FOD814-D, U102 STM32F030F4P6, U103 74HC595, U104 74HC595, U105 LTV-827, U106 IE1203S, U201 TRIAC, U202 TRIAC, U203 TRIAC, U204 TRIAC, U205 TRIAC, U206 TRIAC, U207 TRIAC, U208 TRIAC, U301 TRIAC, U302 TRIAC, U303 TRIAC, U304 TRIAC, U305 TRIAC, U306 TRIAC, U307 TRIAC, U308 TRIAC

Commit message: Should mostly be done.
Needs to be checked over.
Parts:
- removed P104: CONN_01X02, Pin_Headers:Pin_Header_Straight_1x02_Pitch2.54mm
- added J104: Conn_01x02, Connectors_OnShore:OSTTC022162, F.Cu at (77.0, 107.0)
- added J105: Conn_01x02, Connectors_OnShore:OSTTC022162, F.Cu at (178.0, 107.0)
- moved J302 23.2 mm to (147.3, 77.2)
- moved J303 23.2 mm to (157.5, 77.2)
- moved J304 23.2 mm to (167.7, 77.2)
- moved J301 23.2 mm to (137.2, 77.2)
- moved C101 23.1 mm to (133.3, 98.2)
- moved C103 23.1 mm to (133.3, 99.8)
- moved C105 23.1 mm to (133.3, 101.2)
- moved J103 23.1 mm to (131.8, 126.4)
- moved J305 23.1 mm to (137.2, 135.7)
- moved C102 23.1 mm to (119.9, 99.9)
- moved C104 23.1 mm to (118.4, 99.9)
- moved C201 23.1 mm to (89.0, 86.0)
- moved C202 23.1 mm to (96.0, 86.0)
- moved C203 23.1 mm to (103.0, 86.0)
- moved C204 23.1 mm to (110.0, 86.0)
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Connections:
- C101 pad 1: +3V3 -> /+VDD
- C102 pad 1: +3V3 -> /+VDD
- C103 pad 1: +3V3 -> /+VDD
- C104 pad 1: +3V3 -> /+VDD
- C105 pad 1: +3V3 -> /+VDD
- D117 pad 1: /STM_VCC -> /+VDD
- P103 pad 3: /STM_VCC -> /+VDD
- U102 pad 16: +3V3 -> /+VDD
- U102 pad 5: +3V3 -> /+VDD
Routing:
- net AC-N: track 63.4 -> 156.9 mm
- net +3V3: track 0.00 -> 90.7 mm, vias 0 -> 7
- net /GND_IN: track 0.00 -> 81.5 mm, vias 0 -> 2
- net /Shift_~OE: track 0.00 -> 61.3 mm, vias 0 -> 4
- net /Shift_SRCLK: track 0.00 -> 60.2 mm, vias 0 -> 4
- net /Shift_RCLK: track 0.00 -> 59.7 mm, vias 0 -> 4
- net /Shift_~SRCLR: track 0.00 -> 57.1 mm, vias 0 -> 2
- net GND: track 0.00 -> 45.5 mm, vias 0 -> 22
- net Net-(U103-Pad9): track 0.00 -> 41.2 mm
- net AC-H: track 0.00 -> 34.3 mm
- net /Shift_SER: track 0.00 -> 33.9 mm, vias 0 -> 2
- net /+VDD: track 0.00 -> 33.8 mm, vias 0 -> 1
- net /STM_SDA: track 0.00 -> 27.8 mm, vias 0 -> 2
- net /CHAN11: track 1.75 -> 28.7 mm, vias 0 -> 2
- net /I2C_SDA: track 0.00 -> 26.9 mm
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- added copper zone on In1.Cu, net AC-H
- added copper zone on In2.Cu, net AC-N
- added copper zone on B.Cu, net GND
Other:
- board outline added: 106 x 63.5 mm
- board text added: "12V"
- board text added: "3v3 GND"
- board text added: "AC Hot"
- board text added: "AC Neutral"
- board text added: "GND"
- board text added: "I2C AC Line Control David Lenfesty 2018"
- board text added: "Revision A"
- board text added: "SCL SDA GND"
