File: AC-LED-Control/AC-LED-Control.kicad_pcb (KiCad board)
At the start: 4 copper layers, 106 x 63.5 mm, 140 parts, among them J101 Conn_01x03, J102 Conn_01x03, J103 Conn_01x02, J104 Conn_01x02, J105 Conn_01x02, J201 Conn_01x02, J202 Conn_01x02, J203 Conn_01x02, J204 Conn_01x02, J205 Conn_01x02, J206 Conn_01x02, J207 Conn_01x02, J208 Conn_01x02, J301 Conn_01x02, J302 Conn_01x02, J303 Conn_01x02, J304 Conn_01x02, J305 Conn_01x02, J306 Conn_01x02, J307 Conn_01x02, J308 Conn_01x02, P103 CONN_01X04, P105 CONN_01X02, SW101 SW_PUSH, U101 FOD814-D, U102 STM32F030F4P6, U103 74HC595, U104 74HC595, U105 LTV-827, U106 IE1203S, U201 TRIAC, U202 TRIAC, U203 TRIAC, U204 TRIAC, U205 TRIAC, U206 TRIAC, U207 TRIAC, U208 TRIAC, U301 TRIAC, U302 TRIAC, U303 TRIAC, U304 TRIAC, U305 TRIAC, U306 TRIAC, U307 TRIAC, U308 TRIAC

Commit message: Removed diode and fixed some dumb DRC errors.
I had to add some vias where they really weren't needed but whatever.
Parts:
- removed D117: D, Diodes_SMD:D_0603
Connections:
- C101 pad 1: /+VDD -> +3V3
- C102 pad 1: /+VDD -> +3V3
- C103 pad 1: /+VDD -> +3V3
- C104 pad 1: /+VDD -> +3V3
- C105 pad 1: /+VDD -> +3V3
- P103 pad 3: /+VDD -> +3V3
- U102 pad 16: /+VDD -> +3V3
- U102 pad 5: /+VDD -> +3V3
Routing:
- net /+VDD: track 33.8 -> 0.00 mm, vias 1 -> 0
- net AC-N: track 156.9 -> 190.7 mm, vias 0 -> 16
- net +3V3: track 90.7 -> 117.8 mm, vias 7 -> 8
