File: AC-LED-Control/AC-LED-Control.sch (KiCad schematic (older format))
At the start: 50 parts, among them J101 Conn_01x03, J102 Conn_01x03, J103 Conn_01x02, P103 CONN_01X04, P104 CONN_01X02, P105 CONN_01X02, SW101 SW_PUSH, U101 FOD814-D, U102 STM32F030F4P6, U103 74HC595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

Commit message: Changed TRIAC from DPAK part to T0-202-3 part.
Parts:
- P103: footprint Pin_Headers:Pin_Header_Straight_1x04 -> Pin_Headers:Pin_Header_Straight_1x04_Pitch2.54mm
Changed lines of the file:
@@
 F 0 "P103" H 2450 2500 50  0000 C CNN
 F 1 "CONN_01X04" V 2550 2750 50  0000 C CNN
-F 2 "Pin_Headers:Pin_Header_Straight_1x04" H 2450 2750 50  0001 C CNN
+F 2 "Pin_Headers:Pin_Header_Straight_1x04_Pitch2.54mm" H 2450 2750 50  0001 C CNN
 F 3 "" H 2450 2750 50  0000 C CNN
 	1    2450 2750

Commit message: Lots of layout + added a diode.
I realised that the power regulator might need protection from the 3v3
line on the programming header.
Added a diode just in case.
Parts:
- added D117: D, Diodes_SMD:D_0603, symbol D
- added R117, R118, R119, R120, R121, R122, R123, R124: 160, Resistors_SMD:R_0603_HandSoldering, symbol R
Connections:
- net +3V3: now also D117.2 (A); no longer P103.3 (P3)
- net CHAN10: now also R119.2; no longer D106.2 (A)
- net CHAN11: now also R120.2; no longer D108.2 (A)
- net CHAN12: now also R121.2; no longer D110.2 (A)
- net CHAN13: now also R122.2; no longer D112.2 (A)
- net CHAN14: now also R123.2; no longer D114.2 (A)
- net CHAN15: now also R124.2; no longer D116.2 (A)
- net CHAN8: now also R117.2; no longer D102.2 (A)
- net CHAN9: now also R118.2; no longer D104.2 (A)
- new net: D102.2 (A), R117.1
- new net: D104.2 (A), R118.1
- new net: D106.2 (A), R119.1
- new net: D108.2 (A), R120.1
- new net: D110.2 (A), R121.1
- new net: D112.2 (A), R122.1
- new net: D114.2 (A), R123.1
- new net: D116.2 (A), R124.1
- new net STM_VCC: D117.1 (K), P103.3 (P3)
Other:
- moved on the sheet: D101, D103, D105, D107, D109, D111, D113, D115, R107, R108, R109, R110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

Commit message: Should mostly be done.
Needs to be checked over.
Parts:
- removed P104: CONN_01X02, Pin_Headers:Pin_Header_Straight_1x02_Pitch2.54mm, symbol CONN_01X02
- added J104, J105: Conn_01x02, Connectors_OnShore:OSTTC022162, symbol Conn_01x02
Connections:
- net +3V3: no longer C101.1, C102.1, C103.1, C104.1, C105.1, U102.16 (VDD), U102.5 (VDDA)
- net AC-H: now also J104.1 (Pin_1), J105.1 (Pin_1)
- net AC-N: now also J104.2 (Pin_2), J105.2 (Pin_2)
- net STM_VCC renamed +VDD
- net +VDD: now also C101.1, C102.1, C103.1, C104.1, C105.1, U102.16 (VDD), U102.5 (VDDA)
Changed lines of the file:
@@
 Can also be\nUSART
 Wire Wire Line
-	950  1650 1550 1650
+	750  1650 1550 1650
 Wire Wire Line
 	1550 1550 1150 1550
@@
 	1150 1550 1150 1650
 Connection ~ 1150 1650
-$Comp
-L +3V3 #PWR015
-U 1 1 5B465D50
-P 950 1650
-F 0 "#PWR015" H 950 1500 50  0001 C CNN
-F 1 "+3V3" H 950 1790 50  0000 C CNN
-F 2 "" H 950 1650 50  0000 C CNN
-F 3 "" H 950 1650 50  0000 C CNN
-	1    950  1650
-	1    0    0    -1
-$EndComp
 Text Notes 5150 950  0    39   ~ 0
 SERCLK clocks in data from SER\nRCLK transfers data from shift registers\nSRCLR clears shift registers (active low)
@@
 Wire Notes Line
 	650  7500 650  6300
-$Comp
-L CONN_01X02 P104
-U 1 1 5B47C991
-P 7600 4650
-F 0 "P104" H 7550 4800 50  0000 C CNN
-F 1 "CONN_01X02" V 7700 4650 50  0000 C CNN
-F 2 "Pin_Headers:Pin_Header_Straight_1x02_Pitch2.54mm" H 7600 4650 50  0001 C CNN
-F 3 "" H 7600 4650 50  0000 C CNN
-	1    7600 4650
-	1    0    0    -1
-$EndComp
 Wire Wire Line
 	7400 4600 7100 4600
@@
 	9100 3700 9100 5950
 $Comp
-L GND #PWR016
+L GND #PWR015
 U 1 1 5B48AF70
 P 9100 5950
-F 0 "#PWR016" H 9100 5700 50  0001 C CNN
+F 0 "#PWR015" H 9100 5700 50  0001 C CNN
 F 1 "GND" H 9100 5800 50  0000 C CNN
 F 2 "" H 9100 5950 50  0000 C CNN
@@
 	10700 3700 10700 5950
 $Comp
-L GND #PWR017
+L GND #PWR016
 U 1 1 5B48B7DB
 P 10700 5950
-F 0 "#PWR017" H 10700 5700 50  0001 C CNN
+F 0 "#PWR016" H 10700 5700 50  0001 C CNN
 F 1 "GND" H 10700 5800 50  0000 C CNN
 F 2 "" H 10700 5950 50  0000 C CNN
@@
 Need isolation, found this:\nBT136S-600D,118
 $Comp
-L +3V3 #PWR018
+L +3V3 #PWR017
 U 1 1 5B49AE2D
 P 6150 6650
-F 0 "#PWR018" H 6150 6500 50  0001 C CNN
+F 0 "#PWR017" H 6150 6500 50  0001 C CNN
 F 1 "+3V3" H 6150 6790 50  0000 C CNN
 F 2 "" H 6150 6650 50  0000 C CNN
@@
 	6050 6850 6150 6850
 $Comp
-L GND #PWR019
+L GND #PWR018
 U 1 1 5B572609
 P 6150 6950
-F 0 "#PWR019" H 6150 6700 50  0001 C CNN
+F 0 "#PWR018" H 6150 6700 50  0001 C CNN
 F 1 "GND" H 6150 6800 50  0000 C CNN
 F 2 "" H 6150 6950 50  0001 C CNN
@@
 	3450 4450 3450 5650
 $Comp
-L GND #PWR020
+L GND #PWR019
 U 1 1 5B57B922
 P 4500 5450
-F 0 "#PWR020" H 4500 5200 50  0001 C CNN
+F 0 "#PWR019" H 4500 5200 50  0001 C CNN
 F 1 "GND" H 4500 5300 50  0000 C CNN
 F 2 "" H 4500 5450 50  0001 C CNN
@@
 Connection ~ 4050 4600
 $Comp
-L +3V3 #PWR021
+L +3V3 #PWR020
 U 1 1 5B57CBCB
 P 3850 4600
-F 0 "#PWR021" H 3850 4450 50  0001 C CNN
+F 0 "#PWR020" H 3850 4450 50  0001 C CNN
 F 1 "+3V3" H 3850 4740 50  0000 C CNN
 F 2 "" H 3850 4600 50  0001 C CNN
@@
 Text Label 2650 2800 0    60   ~ 0
 STM_VCC
+Text Label 750  1650 0    60   ~ 0
+STM_VCC
+$Comp
+L Conn_01x02 J104
+U 1 1 5B586C53
+P 7600 4600
+F 0 "J104" H 7600 4700 50  0000 C CNN
+F 1 "Conn_01x02" H 7600 4400 50  0000 C CNN
+F 2 "Connectors_OnShore:OSTTC022162" H 7600 4600 50  0001 C CNN
+F 3 "" H 7600 4600 50  0001 C CNN
+	1    7600 4600
+	1    0    0    -1
+$EndComp
+Wire Wire Line
+	7400 5000 7100 5000
+Wire Wire Line
+	7400 5100 7100 5100
+Text GLabel 7100 5000 0    59   Input ~ 0
+AC-H
+Text GLabel 7100 5100 0    59   Input ~ 0
+AC-N
+$Comp
+L Conn_01x02 J105
+U 1 1 5B586EE7
+P 7600 5000
+F 0 "J105" H 7600 5100 50  0000 C CNN
+F 1 "Conn_01x02" H 7600 4800 50  0000 C CNN
+F 2 "Connectors_OnShore:OSTTC022162" H 7600 5000 50  0001 C CNN
+F 3 "" H 7600 5000 50  0001 C CNN
+	1    7600 5000
+	1    0    0    -1
+$EndComp
 $EndSCHEMATC

Commit message: Removed diode and fixed some dumb DRC errors.
I had to add some vias where they really weren't needed but whatever.
Parts:
- removed D117: D, Diodes_SMD:D_0603, symbol D
Connections:
- net +VDD is gone; now on net +3V3: C101.1, C102.1, C103.1, C104.1, C105.1, P103.3 (P3), U102.16 (VDD), U102.5 (VDDA)
Changed lines of the file:
@@
 Can also be\nUSART
-Wire Wire Line
-	750  1650 1550 1650
 Wire Wire Line
 	1550 1550 1150 1550
@@
 Wire Notes Line
 	8000 6200 8650 6200
-$Comp
-L D D117
-U 1 1 5B585061
-P 3150 2800
-F 0 "D117" H 3150 2900 50  0000 C CNN
-F 1 "D" H 3150 2700 50  0000 C CNN
-F 2 "Diodes_SMD:D_0603" H 3150 2800 50  0001 C CNN
-F 3 "" H 3150 2800 50  0001 C CNN
-	1    3150 2800
-	1    0    0    -1
-$EndComp
-Wire Wire Line
-	3000 2800 2650 2800
-Text Label 2650 2800 0    60   ~ 0
-STM_VCC
-Text Label 750  1650 0    60   ~ 0
-STM_VCC
+Wire Wire Line
+	2650 2800 3300 2800
 $Comp
 L Conn_01x02 J104
@@
 	1    0    0    -1
 $EndComp
+$Comp
+L +3V3 #PWR?
+U 1 1 5B5906B7
+P 950 1650
+F 0 "#PWR?" H 950 1500 50  0001 C CNN
+F 1 "+3V3" H 950 1790 50  0000 C CNN
+F 2 "" H 950 1650 50  0000 C CNN
+F 3 "" H 950 1650 50  0000 C CNN
+	1    950  1650
+	1    0    0    -1
+$EndComp
+Wire Wire Line
+	1550 1650 950  1650
 $EndSCHEMATC
