File: 1ch-AC-Control/1ch-AC-Control.kicad_pcb (KiCad board)
At the start: 2 copper layers, 51 x 23 mm, 17 parts, among them J1 Conn_01x02, J2 Conn_01x02, J3 Conn_01x02, J4 Conn_01x03, J5 Conn_01x02, Q1 Q_NMOS_GDSD, U1 LTV-354T, U2 LTV-356T

Commit message: Changed up isolation scheme and added BOM
Instead of isolating each of the TRIAC channels individually,
I changed it so the system uses an isolated power supply and isolates
itself from I2C as well.

Basic BOM was started as well.
Changed lines of the file:
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@@
     (links 26)
     (no_connects 0)
-    (area 130.924999 90.924999 182.075001 114.075001)
+    (area 123.452381 82.45238 190.54762 120.625)
     (thickness 1.6)
     (drawings 15)
@@
     (pad_to_mask_clearance 0.2)
     (aux_axis_origin 0 0)
-    (visible_elements FFFFFF7F)
+    (visible_elements 7FFFFFFF)
     (pcbplotparams
-      (layerselection 0x00030_80000001)
+      (layerselection 0x010f0_80000001)
       (usegerberextensions false)
       (excludeedgelayer true)
@@
       (outputformat 1)
       (mirror false)
-      (drillshape 1)
+      (drillshape 0)
       (scaleselection 1)
-      (outputdirectory ""))
+      (outputdirectory Gerbers/))
   )
   (net 0 "")
@@
       (effects (font (size 1 1) (thickness 0.15)))
     )
-    (fp_text value 1K (at 0 1.75 270) (layer F.Fab)
+    (fp_text value 1K (at -3.35 -0.5 270) (layer F.Fab)
       (effects (font (size 1 1) (thickness 0.15)))
     )
@@
       (effects (font (size 1 1) (thickness 0.15)))
     )
-    (fp_text value 10K (at 0 1.75 90) (layer F.Fab)
+    (fp_text value 10K (at 3.35 0.5 90) (layer F.Fab)
       (effects (font (size 1 1) (thickness 0.15)))
     )
@@
     (effects (font (size 1.5 1.5) (thickness 0.3)))
   )
-  (gr_text Load (at 163 93 360) (layer F.SilkS)
+  (gr_text Load (at 163 93) (layer F.SilkS)
     (effects (font (size 1.5 1.5) (thickness 0.3)))
   )
